File: eagle/tick-ref-gps.brd (EAGLE design)
At the start: 160 x 100 mm, 47 parts, among them CN1 1PPS Out, CN2 ISP, CN3 RS232, CN4 Power In, CN5 Serial Program, U1 ATMEGA168-AU, U2 AS1115, U3 MAX232, U4 LM2931_FIXED, X1 16MHz

Commit message: Routing in progress, 42 airwires left to route.
Parts:
- added JP3: Standalone/PC, SparkFun:SJ_2S-NO
- JP2: device SparkFun:SJ_2S-NO -> SparkFun:1X02_LOCK
- moved TP4 410.6 mm to (83.8, 40.6), flipped to the bottom
- moved TP3 398.3 mm to (73.7, 40.6), flipped to the bottom
- moved TP6 397.1 mm to (27.9, 47.0), flipped to the bottom
- moved TP2 396.6 mm to (53.3, 61.0), flipped to the bottom
- moved TP1 396.3 mm to (63.5, 61.0), flipped to the bottom
- moved C13 392.3 mm to (47.0, 75.2), turned to 90 degrees
- moved TP5 389.3 mm to (25.4, 47.0), flipped to the bottom
- moved C9 373.2 mm to (44.8, 75.2), turned to 90 degrees
- moved C10 351.2 mm to (26.7, 55.9), turned to 90 degrees
- moved C11 343.3 mm to (32.4, 37.1)
- moved C12 342.9 mm to (19.4, 40.6), turned to 90 degrees
- moved R5 338.8 mm to (77.5, 11.4), turned to 180 degrees
- moved CN4 326.5 mm to (66.7, 66.0), flipped to the bottom
- moved LED4 323.8 mm to (72.4, 12.7)
- moved R4 322.4 mm to (59.7, 11.4), turned to 180 degrees
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Connections:
- net 1PPS_RTN: now also CN1.3, CN1.4, CN1.5
- net FTDI_RX-I: now also JP3.1
- net GND: now also GPS1.MOUNT1, GPS1.MOUNT2, GPS1.MOUNT3, GPS1.MOUNT4; no longer CN1.3, CN1.4, CN1.5
- net GPS_RX: now also JP3.2
- net LED_BATT: now also U1.15; no longer U1.16
- net LED_FAULT: now also U1.16; no longer U1.15
- net LED_GPSFIX: now also U1.14; no longer U1.17
Routing:
- net +5V: track 0.00 -> 131.8 mm
- net LED_SEG_G: track 0.00 -> 109.4 mm
- net LED_SEG_F: track 0.00 -> 79.1 mm
- net LED_SEG_C: track 0.00 -> 73.9 mm
- net LED_SEG_B: track 0.00 -> 73.9 mm
- net LED_SEG_A: track 0.00 -> 73.9 mm
- net 1PPS_RTN: track 0.00 -> 68.0 mm
- net LED_FAULT: track 0.00 -> 63.2 mm
- net LED_BATT: track 0.00 -> 47.0 mm
- net LED_SEG_E: track 0.00 -> 41.6 mm
- net 1PPS: track 0.00 -> 37.2 mm
- net FTDI_TX-O: track 0.00 -> 32.9 mm
- net LED_GPSFIX: track 0.00 -> 30.6 mm
- net AVR_RESET: track 0.00 -> 29.8 mm, vias 0 -> 2
- net SDA: track 0.00 -> 28.7 mm
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- added copper zone on layer 1, net GND
- added copper zone on layer 16, net GND
Other:
- board size 160 x 100 mm -> 91.4 x 106.3 mm

Commit message: Completed routing, pending silk and checklist.
Parts:
- moved CN2 58.1 mm to (15.9, 2.54), flipped to the bottom
- moved C1 3.62 mm to (13.7, 38.4), turned to 270 degrees
- moved C2 3.62 mm to (13.7, 35.2), turned to 90 degrees
- moved C12 0.32 mm to (19.1, 40.6)
- moved C9 0.19 mm to (44.8, 75.4)
Connections:
- net ISP_MISO: now also U1.16; no longer U1.2
- net ISP_MOSI: now also U1.15; no longer U1.1
- net ISP_SCK: now also U1.17; no longer U1.9
- net LED_BATT: now also U1.13; no longer U1.15
- net LED_FAULT: now also U1.14; no longer U1.16
- net LED_GPSFIX: now also U1.12; no longer U1.14
Routing:
- net LED_SEG_D: track 0.00 -> 131.4 mm, vias 0 -> 3
- net +5V: track 131.8 -> 234.6 mm, vias 0 -> 6
- net LED_SEG_A: track 73.9 -> 154.8 mm, vias 0 -> 3
- net VBATT: track 0.00 -> 72.1 mm, vias 0 -> 1
- net LED_SEG_F: track 79.1 -> 148.8 mm, vias 0 -> 3
- net LED_SEG_E: track 41.6 -> 110.3 mm, vias 0 -> 1
- net GPS_TX: track 11.1 -> 74.4 mm, vias 0 -> 1
- net LED_SEG_G: track 109.4 -> 172.6 mm, vias 0 -> 3
- net LED_SEG_B: track 73.9 -> 133.3 mm, vias 0 -> 2
- net GPS_RX: track 18.6 -> 72.6 mm, vias 0 -> 2
- net CATH_MIN_LS: track 0.00 -> 52.4 mm, vias 0 -> 4
- net ISP_SCK: track 0.00 -> 51.9 mm, vias 0 -> 1
- net CATH_MIN_MS: track 0.00 -> 50.9 mm, vias 0 -> 4
- net CATH_SEC_LS: track 0.00 -> 49.9 mm, vias 0 -> 2
- net CATH_SEC_MS: track 0.00 -> 48.7 mm, vias 0 -> 2
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
Commit message: Completed routing and silk, still needs final checklist run before CAMing.
Parts:
- added DA1: BAT54C, diode:SOT23
- added LED5: Comms, led:LED5MM
- added R7: 18, rcl:R0603
- added U$1: (no value), logos-sen:OSHW-LOGO-L
- added U$2: (no value), strichlabs:STRICH-LOGO-R
- moved LED2 8.89 mm to (45.7, 12.7)
- moved R6 8.26 mm to (50.2, 11.4)
- moved LED3 6.03 mm to (60.6, 12.7)
- moved R5 5.72 mm to (75.6, 6.03), turned to 0 degrees
- moved R4 5.40 mm to (65.1, 11.4)
- moved R3 3.81 mm to (20.3, 11.4)
- moved LED1 3.18 mm to (15.9, 12.7)
- moved LED4 3.17 mm to (75.6, 12.7)
- moved JP1 1.91 mm to (77.5, 75.6)
- moved BAT1 0.95 mm to (84.5, 26.4)
Connections:
- new net LED5_D: DA1.3, LED5.A
- new net LED5_R: LED5.K, R7.2
- net GND: now also R7.1
- net GPS_RX: now also DA1.1
- net GPS_TX: now also DA1.2
Routing:
- net VBATT: track 72.1 -> 123.4 mm
- net LED5_D: track 0.00 -> 39.4 mm, vias 0 -> 1
- net LED_GPSFIX: track 32.1 -> 40.1 mm
- net GPS_RX: track 72.6 -> 80.2 mm
- net LED_BATT: track 48.6 -> 54.0 mm
- net LED4_R: track 3.49 -> 6.84 mm
- net LED5_R: track 0.00 -> 2.85 mm
- net LED_FAULT: track 65.5 -> 67.8 mm
- net 1PPS_RTN: track 68.0 -> 65.8 mm
- net GPS_TX: track 74.4 -> 76.3 mm
- net ISP_SCK: track 51.9 -> 53.6 mm
- net +5V: track 234.6 -> 235.7 mm
- net LED3_R: track 3.49 -> 2.85 mm
- net LED2_R: track 3.49 -> 2.85 mm
- net LED1_R: track 3.49 -> 2.85 mm
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Other:
- board text added: "+"
- board text added: "-"
- board text added: "1PPS Out"
- board text added: "6-20VDC"
- board text added: "Comms"
- board text added: "Fault"
- board text added: "GPS Fix"
- board text added: "HackLab.TO"
- board text added: "Hour"
- board text added: "ISP"
- board text added: "Minute"
- board text added: "Power"
- board text added: "RS232"
- board text added: "Repl Batt"
- board text added: "Rev001"
- board text added: "Satellites Tracked"
- board text added: "Second"
- board text added: "Serial Program"
- board text added: "UTC"
- board text added: "tick-ref-gps"
