File: eagle/disp/tick-ref-gps-disp.sch (EAGLE design)
At the start: 35 parts, among them CN1 To Main Board, Q1 MMBT3904, U1 AS1115, U2 AS1115

Commit message: Routing continues, 9 airwires to go.
Parts:
- added LED10, LED11, LED12, LED13, LED14, LED15, LED16, LED17, LED18, LED19, LED20, LED21, LED22, LED7, LED8, LED9: (no value), led:LEDCHIP-LED0805
Connections:
- net N$1 renamed 1PPS_R_Q
- removed net CATH_SATS_MS: DSP4.C@1, DSP4.C@2, U2.CATH6
- new net CATH_STATUS_MS: DSP4.C@1, DSP4.C@2, LED21.C, U2.CATH6
- new net CATH_STRENGTH: LED22.C, U2.CATH7
- new net DSPA_SEG_DP: LED15.A, LED16.A, LED17.A, LED18.A, LED19.A, LED20.A, LED21.A, LED22.A, U2.SEGDP
- new net DSPB_SEG_DP: LED10.C, LED11.C, LED12.C, LED13.C, LED14.C, LED7.C, LED8.C, LED9.C, U1.SEGDP
- net CATH_HOUR_LS: now also LED16.C
- net CATH_HOUR_MS: now also LED15.C
- net CATH_MIN_LS: now also LED18.C
- net CATH_MIN_MS: now also LED17.C
- net CATH_SEC_LS: now also LED20.C
- net CATH_SEC_MS: now also LED19.C
- net DSP10-C: now also LED12.A
- net DSP11-C: now also LED13.A
- net DSP12-C: now also LED14.A
- net DSP5-C: now also LED7.A
- net DSP6-C: now also LED8.A
- net DSP7-C: now also LED9.A
- net DSP8-C: now also LED10.A
- net DSP9-C: now also LED11.A
- net DSPB_SEG_G: now also U1.KEYA
Other:
- note added: "SV 1 C/No"
- note added: "SV 2 C/No"
- note added: "SV 3 C/No"
- note added: "SV 4 C/No"
- moved on the sheet: C1, C2, C3, C4, CN1, DSP1, DSP10, DSP11, DSP12, DSP2, DSP3, DSP4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
